Commit message: Loaded darins urdf into mujoco visualizer

File: assets/descriptions/bittle/urdf/bittle.urdf (robot description, URDF)
Before this commit: robot bittle, 87 links, 86 joints
Links:
- link a_1: geometry collision mesh filename=a_1.stl scale=0.001 0.001 0.001; visual mesh filename=a_1.stl scale=0.001 0.001 0.001
- link b__1: geometry collision mesh filename=b__1.stl scale=0.001 0.001 0.001; visual mesh filename=b__1.stl scale=0.001 0.001 0.001
- link base_link: geometry collision mesh filename=base_link.stl scale=0.001 0.001 0.001; visual mesh filename=base_link.stl scale=0.001 0.001 0.001
- link battery_1: geometry collision mesh filename=battery_1.stl scale=0.001 0.001 0.001; visual mesh filename=battery_1.stl scale=0.001 0.001 0.001
- link c_1: geometry collision mesh filename=c_1.stl scale=0.001 0.001 0.001; visual mesh filename=c_1.stl scale=0.001 0.001 0.001
- link c_neck__1: geometry collision mesh filename=c_neck__1.stl scale=0.001 0.001 0.001; visual mesh filename=c_neck__1.stl scale=0.001 0.001 0.001
- link c_thlf_1: geometry collision mesh filename=c_thlf_1.stl scale=0.001 0.001 0.001; visual mesh filename=c_thlf_1.stl scale=0.001 0.001 0.001
- link c_thlr_1: geometry collision mesh filename=c_thlr_1.stl scale=0.001 0.001 0.001; visual mesh filename=c_thlr_1.stl scale=0.001 0.001 0.001
- link c_tholf_1: geometry collision mesh filename=c_tholf_1.stl scale=0.001 0.001 0.001; visual mesh filename=c_tholf_1.stl scale=0.001 0.001 0.001
- link c_tholr__1: geometry collision mesh filename=c_tholr__1.stl scale=0.001 0.001 0.001; visual mesh filename=c_tholr__1.stl scale=0.001 0.001 0.001
- link c_thorf_1: geometry collision mesh filename=c_thorf_1.stl scale=0.001 0.001 0.001; visual mesh filename=c_thorf_1.stl scale=0.001 0.001 0.001
- link c_thorr_1: geometry collision mesh filename=c_thorr_1.stl scale=0.001 0.001 0.001; visual mesh filename=c_thorr_1.stl scale=0.001 0.001 0.001
- link c_thrf__1: geometry collision mesh filename=c_thrf__1.stl scale=0.001 0.001 0.001; visual mesh filename=c_thrf__1.stl scale=0.001 0.001 0.001
- link c_thrr_1: geometry collision mesh filename=c_thrr_1.stl scale=0.001 0.001 0.001; visual mesh filename=c_thrr_1.stl scale=0.001 0.001 0.001
- link cover_1: geometry collision mesh filename=cover_1.stl scale=0.001 0.001 0.001; visual mesh filename=cover_1.stl scale=0.001 0.001 0.001
- link d_1: geometry collision mesh filename=d_1.stl scale=0.001 0.001 0.001; visual mesh filename=d_1.stl scale=0.001 0.001 0.001
- link e_1: geometry collision mesh filename=e_1.stl scale=0.001 0.001 0.001; visual mesh filename=e_1.stl scale=0.001 0.001 0.001
- link f_1: geometry collision mesh filename=f_1.stl scale=0.001 0.001 0.001; visual mesh filename=f_1.stl scale=0.001 0.001 0.001
- link front__1: geometry collision mesh filename=front__1.stl scale=0.001 0.001 0.001; visual mesh filename=front__1.stl scale=0.001 0.001 0.001
- link g_1: geometry collision mesh filename=g_1.stl scale=0.001 0.001 0.001; visual mesh filename=g_1.stl scale=0.001 0.001 0.001
- link h__1: geometry collision mesh filename=h__1.stl scale=0.001 0.001 0.001; visual mesh filename=h__1.stl scale=0.001 0.001 0.001
- link head__1: geometry collision mesh filename=head__1.stl scale=0.001 0.001 0.001; visual mesh filename=head__1.stl scale=0.001 0.001 0.001
- link i_1: geometry collision mesh filename=i_1.stl scale=0.001 0.001 0.001; visual mesh filename=i_1.stl scale=0.001 0.001 0.001
- link j__1: geometry collision mesh filename=j__1.stl scale=0.001 0.001 0.001; visual mesh filename=j__1.stl scale=0.001 0.001 0.001
- link jaw_1: geometry collision mesh filename=jaw_1.stl scale=0.001 0.001 0.001; visual mesh filename=jaw_1.stl scale=0.001 0.001 0.001
- link k_1: geometry collision mesh filename=k_1.stl scale=0.001 0.001 0.001; visual mesh filename=k_1.stl scale=0.001 0.001 0.001
- link l_1: geometry collision mesh filename=l_1.stl scale=0.001 0.001 0.001; visual mesh filename=l_1.stl scale=0.001 0.001 0.001
- link logo_1_1: geometry collision mesh filename=logo_1_1.stl scale=0.001 0.001 0.001; visual mesh filename=logo_1_1.stl scale=0.001 0.001 0.001
- link logo_2_1: geometry collision mesh filename=logo_2_1.stl scale=0.001 0.001 0.001; visual mesh filename=logo_2_1.stl scale=0.001 0.001 0.001
- link logo_3_1: geometry collision mesh filename=logo_3_1.stl scale=0.001 0.001 0.001; visual mesh filename=logo_3_1.stl scale=0.001 0.001 0.001
- link logo_4_1: geometry collision mesh filename=logo_4_1.stl scale=0.001 0.001 0.001; visual mesh filename=logo_4_1.stl scale=0.001 0.001 0.001
- link logo_5_1: geometry collision mesh filename=logo_5_1.stl scale=0.001 0.001 0.001; visual mesh filename=logo_5_1.stl scale=0.001 0.001 0.001
- link rear__1: geometry collision mesh filename=rear__1.stl scale=0.001 0.001 0.001; visual mesh filename=rear__1.stl scale=0.001 0.001 0.001
- link screw_10_1: geometry collision mesh filename=screw_10_1.stl scale=0.001 0.001 0.001; visual mesh filename=screw_10_1.stl scale=0.001 0.001 0.001
- link screw_11_1: geometry collision mesh filename=screw_11_1.stl scale=0.001 0.001 0.001; visual mesh filename=screw_11_1.stl scale=0.001 0.001 0.001
- link screw_12_1: geometry collision mesh filename=screw_12_1.stl scale=0.001 0.001 0.001; visual mesh filename=screw_12_1.stl scale=0.001 0.001 0.001
- link screw_13_1: geometry collision mesh filename=screw_13_1.stl scale=0.001 0.001 0.001; visual mesh filename=screw_13_1.stl scale=0.001 0.001 0.001
- link screw_14_1: geometry collision mesh filename=screw_14_1.stl scale=0.001 0.001 0.001; visual mesh filename=screw_14_1.stl scale=0.001 0.001 0.001
- link screw_15_1: geometry collision mesh filename=screw_15_1.stl scale=0.001 0.001 0.001; visual mesh filename=screw_15_1.stl scale=0.001 0.001 0.001
- link screw_16_1: geometry collision mesh filename=screw_16_1.stl scale=0.001 0.001 0.001; visual mesh filename=screw_16_1.stl scale=0.001 0.001 0.001
- link screw_17_1: geometry collision mesh filename=screw_17_1.stl scale=0.001 0.001 0.001; visual mesh filename=screw_17_1.stl scale=0.001 0.001 0.001
- link screw_18_1: geometry collision mesh filename=screw_18_1.stl scale=0.001 0.001 0.001; visual mesh filename=screw_18_1.stl scale=0.001 0.001 0.001
- link screw_19_1: geometry collision mesh filename=screw_19_1.stl scale=0.001 0.001 0.001; visual mesh filename=screw_19_1.stl scale=0.001 0.001 0.001
- link screw_1_1: geometry collision mesh filename=screw_1_1.stl scale=0.001 0.001 0.001; visual mesh filename=screw_1_1.stl scale=0.001 0.001 0.001
- link screw_20_1: geometry collision mesh filename=screw_20_1.stl scale=0.001 0.001 0.001; visual mesh filename=screw_20_1.stl scale=0.001 0.001 0.001
- link screw_21_1: geometry collision mesh filename=screw_21_1.stl scale=0.001 0.001 0.001; visual mesh filename=screw_21_1.stl scale=0.001 0.001 0.001
- link screw_2_1: geometry collision mesh filename=screw_2_1.stl scale=0.001 0.001 0.001; visual mesh filename=screw_2_1.stl scale=0.001 0.001 0.001
- link screw_3_1: geometry collision mesh filename=screw_3_1.stl scale=0.001 0.001 0.001; visual mesh filename=screw_3_1.stl scale=0.001 0.001 0.001
- link screw_4_1: geometry collision mesh filename=screw_4_1.stl scale=0.001 0.001 0.001; visual mesh filename=screw_4_1.stl scale=0.001 0.001 0.001
- link screw_5_1: geometry collision mesh filename=screw_5_1.stl scale=0.001 0.001 0.001; visual mesh filename=screw_5_1.stl scale=0.001 0.001 0.001
- link screw_6_1: geometry collision mesh filename=screw_6_1.stl scale=0.001 0.001 0.001; visual mesh filename=screw_6_1.stl scale=0.001 0.001 0.001
- link screw_7_1: geometry collision mesh filename=screw_7_1.stl scale=0.001 0.001 0.001; visual mesh filename=screw_7_1.stl scale=0.001 0.001 0.001
- link screw_8_1: geometry collision mesh filename=screw_8_1.stl scale=0.001 0.001 0.001; visual mesh filename=screw_8_1.stl scale=0.001 0.001 0.001
- link screw_9_1: geometry collision mesh filename=screw_9_1.stl scale=0.001 0.001 0.001; visual mesh filename=screw_9_1.stl scale=0.001 0.001 0.001
- link screwm_1_1: geometry collision mesh filename=screwm_1_1.stl scale=0.001 0.001 0.001; visual mesh filename=screwm_1_1.stl scale=0.001 0.001 0.001
- link screwm_2_1: geometry collision mesh filename=screwm_2_1.stl scale=0.001 0.001 0.001; visual mesh filename=screwm_2_1.stl scale=0.001 0.001 0.001
- link screwm_3_1: geometry collision mesh filename=screwm_3_1.stl scale=0.001 0.001 0.001; visual mesh filename=screwm_3_1.stl scale=0.001 0.001 0.001
- link screwm_4_1: geometry collision mesh filename=screwm_4_1.stl scale=0.001 0.001 0.001; visual mesh filename=screwm_4_1.stl scale=0.001 0.001 0.001
- link screwm_5_1: geometry collision mesh filename=screwm_5_1.stl scale=0.001 0.001 0.001; visual mesh filename=screwm_5_1.stl scale=0.001 0.001 0.001
- link screwm_6_1: geometry collision mesh filename=screwm_6_1.stl scale=0.001 0.001 0.001; visual mesh filename=screwm_6_1.stl scale=0.001 0.001 0.001
- link screwm_7_1: geometry collision mesh filename=screwm_7_1.stl scale=0.001 0.001 0.001; visual mesh filename=screwm_7_1.stl scale=0.001 0.001 0.001
- link screwm_8_1: geometry collision mesh filename=screwm_8_1.stl scale=0.001 0.001 0.001; visual mesh filename=screwm_8_1.stl scale=0.001 0.001 0.001
- link servo_lfs_1: geometry collision mesh filename=servo_lfs_1.stl scale=0.001 0.001 0.001; visual mesh filename=servo_lfs_1.stl scale=0.001 0.001 0.001
- link servo_lrs__1: geometry collision mesh filename=servo_lrs__1.stl scale=0.001 0.001 0.001; visual mesh filename=servo_lrs__1.stl scale=0.001 0.001 0.001
- link servo_neck__1: geometry collision mesh filename=servo_neck__1.stl scale=0.001 0.001 0.001; visual mesh filename=servo_neck__1.stl scale=0.001 0.001 0.001
- link servo_rfs_1: geometry collision mesh filename=servo_rfs_1.stl scale=0.001 0.001 0.001; visual mesh filename=servo_rfs_1.stl scale=0.001 0.001 0.001
- link servo_rrs__1: geometry collision mesh filename=servo_rrs__1.stl scale=0.001 0.001 0.001; visual mesh filename=servo_rrs__1.stl scale=0.001 0.001 0.001
- link servos_lf_1: geometry collision mesh filename=servos_lf_1.stl scale=0.001 0.001 0.001; visual mesh filename=servos_lf_1.stl scale=0.001 0.001 0.001
- link servos_lr_1: geometry collision mesh filename=servos_lr_1.stl scale=0.001 0.001 0.001; visual mesh filename=servos_lr_1.stl scale=0.001 0.001 0.001
- link servos_rf_1: geometry collision mesh filename=servos_rf_1.stl scale=0.001 0.001 0.001; visual mesh filename=servos_rf_1.stl scale=0.001 0.001 0.001
- link servos_rr_1: geometry collision mesh filename=servos_rr_1.stl scale=0.001 0.001 0.001; visual mesh filename=servos_rr_1.stl scale=0.001 0.001 0.001
- link shank_lf_1: geometry collision mesh filename=shank_lf_1.stl scale=0.001 0.001 0.001; visual mesh filename=shank_lf_1.stl scale=0.001 0.001 0.001
- link shank_lr_1: geometry collision mesh filename=shank_lr_1.stl scale=0.001 0.001 0.001; visual mesh filename=shank_lr_1.stl scale=0.001 0.001 0.001
- link shank_rf_1: geometry collision mesh filename=shank_rf_1.stl scale=0.001 0.001 0.001; visual mesh filename=shank_rf_1.stl scale=0.001 0.001 0.001
- link shank_rr_1: geometry collision mesh filename=shank_rr_1.stl scale=0.001 0.001 0.001; visual mesh filename=shank_rr_1.stl scale=0.001 0.001 0.001
- link th_lf_1: geometry collision mesh filename=th_lf_1.stl scale=0.001 0.001 0.001; visual mesh filename=th_lf_1.stl scale=0.001 0.001 0.001
- link th_lr__1: geometry collision mesh filename=th_lr__1.stl scale=0.001 0.001 0.001; visual mesh filename=th_lr__1.stl scale=0.001 0.001 0.001
- link th_rf_1: geometry collision mesh filename=th_rf_1.stl scale=0.001 0.001 0.001; visual mesh filename=th_rf_1.stl scale=0.001 0.001 0.001
- link th_rr_1: geometry collision mesh filename=th_rr_1.stl scale=0.001 0.001 0.001; visual mesh filename=th_rr_1.stl scale=0.001 0.001 0.001
- link tho_lf_1: geometry collision mesh filename=tho_lf_1.stl scale=0.001 0.001 0.001; visual mesh filename=tho_lf_1.stl scale=0.001 0.001 0.001
- link tho_lr_1: geometry collision mesh filename=tho_lr_1.stl scale=0.001 0.001 0.001; visual mesh filename=tho_lr_1.stl scale=0.001 0.001 0.001
- link tho_rf__1: geometry collision mesh filename=tho_rf__1.stl scale=0.001 0.001 0.001; visual mesh filename=tho_rf__1.stl scale=0.001 0.001 0.001
- link tho_rr_1: geometry collision mesh filename=tho_rr_1.stl scale=0.001 0.001 0.001; visual mesh filename=tho_rr_1.stl scale=0.001 0.001 0.001
- link tube__1: geometry collision mesh filename=tube__1.stl scale=0.001 0.001 0.001; visual mesh filename=tube__1.stl scale=0.001 0.001 0.001
- link tube_lf_1: geometry collision mesh filename=tube_lf_1.stl scale=0.001 0.001 0.001; visual mesh filename=tube_lf_1.stl scale=0.001 0.001 0.001
- link tube_lr_1: geometry collision mesh filename=tube_lr_1.stl scale=0.001 0.001 0.001; visual mesh filename=tube_lr_1.stl scale=0.001 0.001 0.001
- link tube_rr_1: geometry collision mesh filename=tube_rr_1.stl scale=0.001 0.001 0.001; visual mesh filename=tube_rr_1.stl scale=0.001 0.001 0.001

File: assets/descriptions/bittle/xacro/bittle.xacro (robot description, xacro)
@@ -1,7 +1,7 @@
 <?xml version="1.0" ?>
 <robot name="bittle" xmlns:xacro="http://www.ros.org/wiki/xacro">
-<xacro:include filename="$(find bittle_description)/urdf/materials.xacro" />
-<xacro:include filename="$(find bittle_description)/urdf/bittle.trans" />
-<xacro:include filename="$(find bittle_description)/urdf/bittle.gazebo" />
+<xacro:include filename="materials.xacro" />
+<xacro:include filename="bittle.trans" />
+<xacro:include filename="bittle.gazebo" />
 <link name="base_link">
   <inertial>

Commit message: parsed mesh zip & updated urdf to use collision meshes

File: assets/descriptions/bittle/urdf/bittle.urdf (robot description, URDF)
Before this commit: robot bittle, 87 links, 86 joints
Links:
- link shank_lf_1: geometry collision mesh filename=shank_lf_1_convex.stl scale=0.001 0.001 0.001; visual mesh filename=shank_lf_1.stl scale=0.001 0.001 0.001
- link shank_lr_1: geometry collision mesh filename=shank_lr_1_convex.stl scale=0.001 0.001 0.001; visual mesh filename=shank_lr_1.stl scale=0.001 0.001 0.001
- link shank_rf_1: geometry collision mesh filename=shank_rf_1_convex.stl scale=0.001 0.001 0.001; visual mesh filename=shank_rf_1.stl scale=0.001 0.001 0.001
- link shank_rr_1: geometry collision mesh filename=shank_rr_1_convex.stl scale=0.001 0.001 0.001; visual mesh filename=shank_rr_1.stl scale=0.001 0.001 0.001
